Commit message: Update trial.urdf

File: urdf/trial.urdf (robot description, URDF)
Before this commit: robot myfirst, 1 links, 0 joints
Links:
- link base_link: geometry visual box size=1.2 0.3 1.2

Commit message: simplified mars rover urdf with 2 joints one for swerve and one to drive

File: urdf/trial.urdf (robot description, URDF)
Before this commit: robot myfirst, 5 links, 4 joints
Joints:
- joint base_to_fl: origin xyz=0.535 0.595 -0.255 rpy=1.57075 0 1.57075 -> xyz=0.535 0.495 -0.255 rpy=1.57075 0 1.57075
