Commit message: updated with collisions and inertias for each component

File: urdf/marsrover.urdf (robot description, URDF)
Before this commit: robot myfirst, 9 links, 8 joints
Links:
- link back_left_wheel: mass None -> 2; geometry collision cylinder length=0.13 radius=0.105; visual cylinder length=0.13 radius=0.105
- link back_right_wheel: mass None -> 2; geometry collision cylinder length=0.13 radius=0.105; visual cylinder length=0.13 radius=0.105
- link base_link: mass None -> 40; geometry collision box size=1.2 1.2 0.3; visual box size=1.2 1.2 0.3
- link block_bl: mass None -> 0.5; geometry collision box size=0.1 0.1 0.1; visual box size=0.1 0.1 0.1
- link block_br: mass None -> 0.5; geometry collision box size=0.1 0.1 0.1; visual box size=0.1 0.1 0.1
- link block_fl: mass None -> 0.5; geometry collision box size=0.1 0.1 0.1; visual box size=0.1 0.1 0.1
- link block_fr: mass None -> 0.5; geometry collision box size=0.1 0.1 0.1; visual box size=0.1 0.1 0.1
- link front_left_wheel: mass None -> 2; geometry collision cylinder length=0.13 radius=0.105; visual cylinder length=0.13 radius=0.105
- link front_right_wheel: mass None -> 2; geometry collision cylinder length=0.13 radius=0.105; visual cylinder length=0.13 radius=0.105
